File: 4ch Mixer.kicad_pcb (KiCad board)
At the start: 2 copper layers, 42 parts, among them J1 JACK_2P, J2 JACK_2P, J3 JACK_2P, J4 JACK_2P, J5 JACK_2P, J6 JACK_2P, P1 CONN_02X08, U1 TL074, U2 TL072

Commit message: Continued work on PCB and Schematic
Parts:
- C1, C2, C3, C4: footprint Capacitors_THT:C_Rect_L11.0mm_W3.4mm_P10.00mm_MKT -> Capacitors_THT:C_Axial_L5.1mm_D3.1mm_P10.00mm_Horizontal
- C5, C6: footprint Capacitors_THT:CP_Radial_D10.0mm_P7.50mm -> Capacitors_THT:CP_Radial_D8.0mm_P5.00mm
- D1, D2: footprint Diodes_THT:D_DO-15_P12.70mm_Horizontal -> Diodes_THT:D_DO-35_SOD27_P2.54mm_Vertical_AnodeUp
- J1, J2, J3, J4, J5, J6: value JACK_2P -> 3.5mm_Mono_Jack_With_Switch; footprint Connectors:JACK_ALIM -> _NTSFootprints:3.5mm_Mono_Vertical_QuingPu_WQP-PJ301M-12
- R1, R10, R11, R12, R13, R14, R15, R16, R17, R18, R19, R2, R3, R4, R5, R6, R7, R8, R9: footprint Resistors_THT:R_Axial_DIN0309_L9.0mm_D3.2mm_P12.70mm_Horizontal -> Resistors_THT:R_Axial_DIN0207_L6.3mm_D2.5mm_P2.54mm_Vertical
- moved P1 160.7 mm to (87.6, 55.9)
- moved J1 138.1 mm to (77.5, 59.7), turned to 270 degrees
- moved J2 135.1 mm to (77.5, 80.0), turned to 270 degrees
- moved J3 132.5 mm to (77.5, 100.3), turned to 270 degrees
- moved J4 130.7 mm to (77.5, 120.7), turned to 270 degrees
- moved C6 109.5 mm to (86.4, 105.4)
- moved C5 104.8 mm to (91.4, 96.5), turned to 180 degrees
- moved J5 95.4 mm to (128.3, 100.3), turned to 90 degrees
- moved J6 94.4 mm to (128.3, 121.9), turned to 90 degrees
- moved D2 87.6 mm to (87.6, 85.1)
- moved D1 82.9 mm to (90.2, 88.9), turned to 180 degrees
- moved U1 82.0 mm to (118.1, 62.2)
- moved F2 79.1 mm to (86.4, 81.3)
- moved F1 77.8 mm to (91.4, 77.5), turned to 180 degrees
- moved U2 70.4 mm to (118.1, 82.5)
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Connections:
- J1 pad 1: Net-(J1-Pad1) -> GNDA
- J1 pad 3: GNDA -> Net-(J1-Pad3)
- J2 pad 1: Net-(J2-Pad1) -> GNDA
- J2 pad 3: GNDA -> Net-(J2-Pad3)
- J3 pad 1: Net-(J3-Pad1) -> GNDA
- J3 pad 3: GNDA -> Net-(J3-Pad3)
- J4 pad 1: Net-(J4-Pad1) -> GNDA
- J4 pad 3: GNDA -> Net-(J4-Pad3)
- J5 pad 1: Net-(J5-Pad1) -> GNDA
- J5 pad 3: GNDA -> Net-(J5-Pad3)
- J6 pad 1: Net-(J6-Pad1) -> GNDA
- J6 pad 3: GNDA -> Net-(J6-Pad3)
- R18 pad 1: Net-(J5-Pad1) -> Net-(J5-Pad3)
- R19 pad 1: Net-(J6-Pad1) -> Net-(J6-Pad3)
- RV1 pad 1: Net-(J1-Pad1) -> Net-(J1-Pad3)
- RV2 pad 1: Net-(J2-Pad1) -> Net-(J2-Pad3)
- RV3 pad 1: Net-(J3-Pad1) -> Net-(J3-Pad3)
- RV4 pad 1: Net-(J4-Pad1) -> Net-(J4-Pad3)

Commit message: Worked on the PCB
Parts:
- moved C5 40.7 mm to (132.1, 97.8)
- moved C6 37.6 mm to (123.2, 97.8), turned to 180 degrees
- moved P1 21.6 mm to (71.1, 69.8), turned to 90 degrees
- moved D2 18.5 mm to (92.7, 67.3), turned to 270 degrees
- moved D1 16.7 mm to (92.7, 72.4), turned to 0 degrees
- moved F1 13.3 mm to (78.7, 73.7)
- moved J5 12.5 mm to (123.2, 111.8)
- moved R16 12.5 mm to (124.5, 105.4)
- moved R18 12.5 mm to (119.4, 105.4)
- moved R14 12.0 mm to (132.1, 90.2)
- moved F2 8.03 mm to (83.8, 73.7)
- moved J6 5.68 mm to (123.2, 124.5)
- moved R17 5.68 mm to (124.5, 118.1)
- moved R19 5.68 mm to (119.4, 118.1)
- moved C3 3.81 mm to (114.3, 97.8)
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Routing:
- net +12VA: track 0.00 -> 79.1 mm
- net -12VA: track 0.00 -> 48.0 mm
- net Net-(J4-Pad3): track 0.00 -> 25.7 mm
- net Net-(J1-Pad3): track 0.00 -> 25.7 mm
- net Net-(J3-Pad3): track 0.00 -> 25.7 mm
- net Net-(J2-Pad3): track 0.00 -> 25.7 mm
- net Net-(F2-Pad1): track 0.00 -> 9.20 mm
- net Net-(R3-Pad1): track 0.00 -> 8.45 mm
- net Net-(R4-Pad1): track 0.00 -> 8.45 mm
- net Net-(R2-Pad1): track 0.00 -> 8.45 mm
- net Net-(R1-Pad1): track 0.00 -> 8.45 mm
- net Net-(R14-Pad1): track 0.00 -> 7.40 mm
- net Net-(J5-Pad3): track 0.00 -> 6.81 mm
- net Net-(J6-Pad3): track 0.00 -> 6.81 mm
- net Net-(R5-Pad2): track 0.00 -> 6.35 mm
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
Commit message: Created PCB.  Need to look over carefully.
Need to measure potentiometer footprint to ensure it is correct.
Parts:
- added D3: LED, LEDs:LED_D3.0mm, F.Cu at (169.9, 54.9)
- added R20: 1k, Resistors_THT:R_Axial_DIN0207_L6.3mm_D2.5mm_P2.54mm_Vertical, F.Cu at (161.0, 54.9)
- moved P1 72.6 mm to (136.9, 100.6), turned to 180 degrees
- moved C4 64.3 mm to (173.7, 99.3), turned to 180 degrees
- moved F1 64.2 mm to (134.4, 105.7), turned to 270 degrees
- moved C3 59.5 mm to (173.7, 95.5), turned to 180 degrees
- moved D1 58.4 mm to (134.4, 113.3), turned to 270 degrees
- moved F2 50.8 mm to (134.4, 79.0), turned to 90 degrees
- moved J5 49.3 mm to (172.5, 112.0)
- moved J6 49.3 mm to (172.5, 124.7)
- moved R18 49.3 mm to (168.7, 105.7)
- moved R19 49.3 mm to (168.7, 118.4)
- moved R16 49.3 mm to (173.7, 105.7)
- moved R17 49.3 mm to (173.7, 118.4)
- moved R15 46.8 mm to (176.3, 86.6)
- moved R3 46.8 mm to (176.3, 73.9)
- moved R4 46.8 mm to (176.3, 68.8)
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Connections:
- P1 pad 2: Net-(P1-Pad1) -> Net-(P1-Pad2)
- P1 pad 4: Net-(P1-Pad3) -> Net-(P1-Pad4)
- P1 pad 6: Net-(P1-Pad5) -> Net-(P1-Pad6)
Routing:
- net -12VA: track 48.0 -> 141.7 mm
- net +12VA: track 79.1 -> 154.0 mm
- net Net-(RV4-Pad2): track 0.00 -> 69.8 mm
- net Net-(R10-Pad1): track 3.81 -> 66.3 mm
- net Net-(RV3-Pad2): track 0.00 -> 58.9 mm
- net Net-(R13-Pad1): track 6.35 -> 48.8 mm
- net Net-(RV2-Pad2): track 0.00 -> 23.3 mm
- net Net-(F1-Pad1): track 6.35 -> 27.3 mm
- net Net-(R15-Pad1): track 6.35 -> 26.5 mm
- net Net-(RV1-Pad2): track 0.00 -> 17.9 mm
- net Net-(D3-Pad2): track 0.00 -> 6.35 mm
- net Net-(F2-Pad1): track 9.20 -> 6.35 mm
- net Net-(P1-Pad5): track 2.54 -> 0.00 mm
- net Net-(P1-Pad3): track 2.54 -> 0.00 mm
- net Net-(P1-Pad1): track 2.54 -> 0.00 mm
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- added copper zone on B.Cu, net GNDA
- added copper zone on F.Cu, net GNDA
Other:
- board outline added: 66 x 80 mm
