File: Faceplate/4ch Mixer Faceplate.kicad_pcb (KiCad board)
At the start: 2 copper layers, 30.5 x 128.5 mm, 15 parts

Commit message: Add module title and output polarity symbols to the front panel
Title 'Quad Mixer' at the Attenuverter's size, italic, centred 7.85 mm below
the top edge. + to the left of the non-inverting output J5 and - to the right
of the inverting output J6. Also hides the placeholder reference on the logo.
DRC: no errors.
Other:
- board text added: "+"
- board text added: "-"
- board text added: "Quad Mixer"
Changed lines of the file:
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@@
+		)
+	)
+	(gr_text "Quad Mixer"
+		(at 115.0 43.6 0)
+		(layer "F.SilkS")
+		(effects
+			(font italic
+				(size 2.5 2.5)
+				(thickness 0.3)
+			)
+		)
+	)
+	(gr_text "+"
+		(at 101.527 145.0 0)
+		(layer "F.SilkS")
+		(effects
+			(font
+				(size 2.0 2.0)
+				(thickness 0.3)
+			)
+		)
+	)
+	(gr_text "-"
+		(at 128.55 145.0 0)
+		(layer "F.SilkS")
+		(effects
+			(font
+				(size 2.0 2.0)
+				(thickness 0.3)
+			)
 		)
 	)
@@
 				)
 			)
+			(hide yes)
 		)
 		(property "Value" ""
