File: Schematic/4ch Mixer.kicad_sch (KiCad schematic)
At the start: 46 parts, among them J1 3.5mm_Mono_Jack_With_Switch, J2 3.5mm_Mono_Jack_With_Switch, J3 3.5mm_Mono_Jack_With_Switch, J4 3.5mm_Mono_Jack_With_Switch, J5 3.5mm_Mono_Jack_With_Switch, J6 3.5mm_Mono_Jack_With_Switch, P1 CONN_02X08, U1 TL074, U2 TL072

Commit message: Remove power LED and its series resistor
The LED indicator is not needed. Removes D3, R20 and their +12VA and
GNDA power symbols.
Parts:
- removed D3: LED, LED_THT:LED_D3.0mm, symbol 4ch-Mixer-rescue:LED
- removed R20: 1k, Resistor_THT:R_Axial_DIN0207_L6.3mm_D2.5mm_P2.54mm_Vertical, symbol 4ch-Mixer-rescue:R

Commit message: Ground input jack sleeves and switch contacts
Pin 1 (sleeve) and pin 2 (switch) of J1-J4 and the R1-R4 input resistor
ends are now tied to GNDA. Adds one GNDA symbol per channel at the
junction corner.
Connections:
- net GNDA: now also J1.1, J1.2, J2.1, J2.2, J3.1, J3.2, J4.1, J4.2, R1.2, R2.2, R3.2, R4.2

Commit message: Use Attenuverter footprints and 10-pin shrouded header
Assign 0805 passives, SOIC op amps, 1206 fuses, SMA diodes, electrolytic
caps, NTS jack/pot footprints and the shrouded 2x05 header. Header pinout
matches the Attenuverter: -12V on pins 1-2, GND on 3-8, +12V on 9-10.
Power symbol names and jack symbol pins are unchanged for now.
Parts:
- removed P1: CONN_02X08, Connector_PinHeader_2.54mm:PinHeader_2x08_P2.54mm_Vertical, symbol 4ch-Mixer-rescue:CONN_02X08
- added P1: Power, symbol Connector_Generic:Conn_02x05_Odd_Even
- C1, C2, C3, C4: footprint Capacitor_THT:C_Axial_L5.1mm_D3.1mm_P10.00mm_Horizontal -> Capacitor_SMD:C_0805_2012Metric
- C5, C6: footprint Capacitor_THT:CP_Radial_D8.0mm_P5.00mm -> Capacitor_SMD:CP_Elec_6.3x5.4
- C7, C8: footprint Capacitor_THT:C_Disc_D3.0mm_W2.0mm_P2.50mm -> Capacitor_SMD:C_0805_2012Metric
- D1, D2: footprint Diode_THT:D_DO-35_SOD27_P2.54mm_Vertical_AnodeUp -> Diode_SMD:D_SMA
- F1, F2: footprint Capacitor_THT:C_Disc_D5.0mm_W2.5mm_P5.00mm -> Fuse:Fuse_1206_3216Metric
- J1, J2, J3, J4, J5, J6: footprint _NTSFootprints:3.5mm_Mono_Vertical_QuingPu_WQP-PJ301M-12 -> _NTSFootprints:Jack_3.5mm_QingPu_WQP-PJ398SM_Vertical_CenterHole_OvalPads
- R1, R10, R11, R12, R13, R14, R15, R16, R17, R18, R19, R2, R3, R4, R5, R6, R7, R8, R9: footprint Resistor_THT:R_Axial_DIN0207_L6.3mm_D2.5mm_P2.54mm_Vertical -> Resistor_SMD:R_0805_2012Metric
- RV1, RV2, RV3, RV4: footprint Potentiometer_THT:Potentiometer_Alps_RK09L_Single_Horizontal -> _NTSFootprints:Potentiometer_Alps_RK09L_Plated_Mount_Holes
- U1: footprint Package_DIP:DIP-14_W7.62mm_Socket -> Package_SO:SOIC-14_3.9x8.7mm_P1.27mm
- U2: footprint Package_DIP:DIP-8_W7.62mm_Socket -> Package_SO:SOIC-8_3.9x4.9mm_P1.27mm
Connections:
- net GNDA: now also P1.3 (Pin_3), P1.4 (Pin_4), P1.5 (Pin_5), P1.6 (Pin_6), P1.7 (Pin_7), P1.8 (Pin_8)
- net at F2.1: now also P1.1 (Pin_1), P1.2 (Pin_2)
- net at F1.1: now also P1.10 (Pin_10), P1.9 (Pin_9)
- no-connect marks 8 -> 2

Commit message: Use AudioJack2_SwitchT for the input and output jacks
Pins renamed to S (sleeve), T (tip) and TN (switch) to match the
PJ398SM footprint pads. Sleeves and input switch contacts stay on GNDA,
tips keep their signal nets. Output switch contacts are unused.
Parts:
- removed J1, J2, J3, J4, J5, J6: 3.5mm_Mono_Jack_With_Switch, _NTSFootprints:Jack_3.5mm_QingPu_WQP-PJ398SM_Vertical_CenterHole_OvalPads, symbol 4ch-Mixer-rescue:3.5mm_Mono_Jack_With_Switch
- added J1, J2, J3, J4, J5, J6: (no value), symbol Connector_Audio:AudioJack2_SwitchT
Connections:
- net GNDA: now also J1.S, J1.TN, J2.S, J2.TN, J3.S, J3.TN, J4.S, J4.TN, J5.S, J6.S
- net at RV1.1: now also J1.T
- net at RV2.1: now also J2.T
- net at RV3.1: now also J3.T
- net at RV4.1: now also J4.T
- net at R18.1: now also J5.T
- net at R19.1: now also J6.T

Commit message: Restore Attenuverter footprints on jacks and header
Changing the jack and header symbols cleared their footprint fields.
Reassign PJ398SM to J1-J6 and the shrouded 2x05 header to P1, then
regenerate the board placement from the updated netlist.
Parts:
- J1, J2, J3, J4, J5, J6: footprint (none) -> _NTSFootprints:Jack_3.5mm_QingPu_WQP-PJ398SM_Vertical_CenterHole_OvalPads
- P1: footprint (none) -> _NTSFootprints:PinHeader_2x05_P2.54mm_Vertical_Shrouded
Changed lines of the file:
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@@
 			)
 		)
-		(property "Footprint" ""
+		(property "Footprint" "_NTSFootprints:Jack_3.5mm_QingPu_WQP-PJ398SM_Vertical_CenterHole_OvalPads"
 			(at 38.1 106.68 0)
 			(hide yes)
@@
 			)
 		)
-		(property "Footprint" ""
+		(property "Footprint" "_NTSFootprints:Jack_3.5mm_QingPu_WQP-PJ398SM_Vertical_CenterHole_OvalPads"
 			(at 236.22 129.54 0)
 			(hide yes)
@@
 			)
 		)
-		(property "Footprint" ""
+		(property "Footprint" "_NTSFootprints:Jack_3.5mm_QingPu_WQP-PJ398SM_Vertical_CenterHole_OvalPads"
 			(at 38.1 30.48 0)
 			(hide yes)
@@
 			)
 		)
-		(property "Footprint" ""
+		(property "Footprint" "_NTSFootprints:Jack_3.5mm_QingPu_WQP-PJ398SM_Vertical_CenterHole_OvalPads"
 			(at 38.1 68.58 0)
 			(hide yes)
@@
 			)
 		)
-		(property "Footprint" ""
+		(property "Footprint" "_NTSFootprints:PinHeader_2x05_P2.54mm_Vertical_Shrouded"
 			(at 233.68 50.8 0)
 			(hide yes)
@@
 			)
 		)
-		(property "Footprint" ""
+		(property "Footprint" "_NTSFootprints:Jack_3.5mm_QingPu_WQP-PJ398SM_Vertical_CenterHole_OvalPads"
 			(at 236.22 99.06 0)
 			(hide yes)
@@
 			)
 		)
-		(property "Footprint" ""
+		(property "Footprint" "_NTSFootprints:Jack_3.5mm_QingPu_WQP-PJ398SM_Vertical_CenterHole_OvalPads"
 			(at 38.1 146.05 0)
 			(hide yes)

Commit message: Routed SMD board
Hand-arranged placement and routing from KiCad, with the schematic missing
connections fixed by hand. The jack footprint uses the Attenuverter's
orientation. DRC: no unconnected items; only the three accepted thermal
spoke warnings remain.
Parts:
- removed C5, C6: 100uf, Capacitor_SMD:CP_Elec_6.3x5.4, symbol 4ch-Mixer-rescue:CP
- added C5, C6: 10uf, Capacitor_SMD:C_0805_2012Metric, symbol 4ch-Mixer-rescue:C
Connections:
- net +12VA: now also C1.1, D1.1 (K), F1.2, C5.1
- net -12VA: now also C6.2
- net GNDA: now also C1.2, C2.1, C3.2, C4.1, D1.2 (A), D2.1 (K), C5.2, C6.1
- net at R5.2, U1.1: now also R9.2; no longer R9.1
- net at C7.2, U2.2 (-): now also R10.1, R11.1, R12.1, R13.2, R9.1
Other:
- moved on the sheet: R9

Commit message: Add input clamp protection and Schentronics logo footprints
Schematic: 1N4148 clamps and 1k series resistors on the inputs.
Library: all four Schentronics logo variants from NTSFootprints.
Parts:
- added D10, D3, D4, D5, D6, D7, D8, D9: 1N4148, Diode_SMD:D_SOD-323, symbol 4ch-Mixer-rescue:D
- added R20, R21, R22, R23: 1k, Resistor_SMD:R_0805_2012Metric, symbol 4ch-Mixer-rescue:R
- R18, R19: value 100 -> 1k
Connections:
- net +12VA: now also D3.1 (K), D5.1 (K), D7.1 (K), D9.1 (K)
- net -12VA: now also D10.2 (A), D4.2 (A), D6.2 (A), D8.2 (A)
- net at U1.3 (+): now also D3.2 (A), D4.1 (K), R20.1; no longer RV1.2
- net at U1.5 (+): now also D5.2 (A), D6.1 (K), R21.1; no longer RV2.2
- net at U1.10 (+): now also D7.2 (A), D8.1 (K), R22.1; no longer RV3.2
- net at U1.12 (+): now also D10.1 (K), D9.2 (A), R23.1; no longer RV4.2
- new net: R20.2, RV1.2
- new net: R21.2, RV2.2
- new net: R22.2, RV3.2
- new net: R23.2, RV4.2
Other:
- moved on the sheet: J1, J2, J3, J4, RV1, RV2, RV3, RV4

Commit message: Add manufacturing files and set rail diodes to MRA4003T3G
Manufacturing: Gerbers and drill for the mixer PCB and front panel, BOMs
(SMD for the fab, hand assembly), and placement files. Schematic: D1 and D2
changed to MRA4003T3G to match the fab BOM.
Parts:
- D1, D2: value 1N4002 -> MRA4003T3G
- F1, F2: value 250mA -> 200mA
Changed lines of the file:
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@@
 			)
 		)
-		(property "Value" "1N4002"
+		(property "Value" "MRA4003T3G"
 			(at 193.04 41.91 0)
 			(show_name no)
@@
 			)
 		)
-		(property "Value" "1N4002"
+		(property "Value" "MRA4003T3G"
 			(at 193.04 55.88 0)
 			(show_name no)
@@
 			)
 		)
-		(property "Value" "250mA"
+		(property "Value" "200mA"
 			(at 205.74 35.56 90)
 			(show_name no)
@@
 			)
 		)
-		(property "Value" "250mA"
+		(property "Value" "200mA"
 			(at 205.74 68.58 90)
 			(show_name no)
