File: hardware/mixer/4ch Mixer.kicad_pcb (KiCad board)
At the start: 2 copper layers, 30 x 100 mm, 60 parts, among them P1 Power, U1 TL074, U2 TL072

Commit message: Swap + and - output positions on the panel; trim pot ring at the edge
Board: J5 (non-inverting, +) is on the right and J6 (inverting, -) on the left,
after the designator and net swap. Panel: + to the right of the J5 hole, -
to the left of the J6 hole. Pot outer rings are cut at the panel edge.
Parts:
- D1, D2: value 1N4002 -> MRA4003T3G
- F1, F2: value 250mA -> 200mA
- renumbered J6 to J5, J5 to J6, R17 to R16, R16 to R17, R19 to R18, R18 to R19
Connections:
- R16 pad 1: Net-(U2A-~) -> Net-(U2B-~)
- R17 pad 1: Net-(U2B-~) -> Net-(U2A-~)
- R18 pad 2: Net-(U2A-~) -> Net-(U2B-~)
- R19 pad 2: Net-(U2B-~) -> Net-(U2A-~)
- RV1 pad : GNDA -> (no net)
- RV2 pad : GNDA -> (no net)
- RV3 pad : GNDA -> (no net)
- RV4 pad : GNDA -> (no net)
Routing:
- net Net-(U2A-~): track 89.3 -> 81.8 mm
- net Net-(U2B-~): track 55.5 -> 60.3 mm
Changed lines of the file:
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@@
 			(layers "*.Cu" "*.Mask")
 			(remove_unused_layers no)
-			(net "GNDA")
 		)
 		(pad "" thru_hole circle
@@
 			(layers "*.Cu" "*.Mask")
 			(remove_unused_layers no)
-			(net "GNDA")
 		)
 		(pad "1" thru_hole circle
@@
 		(descr "TRS 3.5mm, vertical, Thonkiconn, PCB mount, (http://www.qingpu-electronics.com/en/products/WQP-PJ398SM-362.html)")
 		(tags "WQP-PJ398SM WQP-PJ301M-12 TRS 3.5mm mono vertical jack thonkiconn qingpu")
-		(property "Reference" "J6"
+		(property "Reference" "J5"
 			(at 4 1.077 0)
 			(layer "F.SilkS")
@@
 		)
 		(fp_text user "KEEPOUT"
-			(at 0 6.48 180)
+			(at 0 6.48 0)
 			(layer "Cmts.User")
 			(effects
@@
 			(layers "*.Cu" "*.Mask")
 			(remove_unused_layers no)
-			(net "Net-(J6-PadT)")
+			(net "Net-(J5-PadT)")
 			(pintype "passive")
 		)
@@
 			(layers "*.Cu" "*.Mask")
 			(remove_unused_layers no)
-			(net "unconnected-(J6-PadTN)")
+			(net "unconnected-(J5-PadTN)")
 			(pintype "passive+no_connect")
 		)
@@
 		(descr "TRS 3.5mm, vertical, Thonkiconn, PCB mount, (http://www.qingpu-electronics.com/en/products/WQP-PJ398SM-362.html)")
 		(tags "WQP-PJ398SM WQP-PJ301M-12 TRS 3.5mm mono vertical jack thonkiconn qingpu")
-		(property "Reference" "J5"
+		(property "Reference" "J6"
 			(at -4.03 1.08 180)
 			(layer "F.SilkS")
@@
 			(layers "*.Cu" "*.Mask")
 			(remove_unused_layers no)
-			(net "Net-(J5-PadT)")
+			(net "Net-(J6-PadT)")
 			(pintype "passive")
 		)
@@
 			(layers "*.Cu" "*.Mask")
 			(remove_unused_layers no)
-			(net "unconnected-(J5-PadTN)")
+			(net "unconnected-(J6-PadTN)")
 			(pintype "passive+no_connect")
 		)
@@
 			(layers "*.Cu" "*.Mask")
 			(remove_unused_layers no)
-			(net "GNDA")
 		)
 		(pad "" thru_hole circle
@@
 			(layers "*.Cu" "*.Mask")
 			(remove_unused_layers no)
-			(net "GNDA")
 		)
 		(pad "1" thru_hole circle
@@
 			(layers "*.Cu" "*.Mask")
 			(remove_unused_layers no)
-			(net "GNDA")
 		)
 		(pad "" thru_hole circle
@@
 			(layers "*.Cu" "*.Mask")
 			(remove_unused_layers no)
-			(net "GNDA")
 		)
 		(pad "1" thru_hole circle
@@
 			(layers "*.Cu" "*.Mask")
 			(remove_unused_layers no)
-			(net "GNDA")
 		)
 		(pad "" thru_hole circle
@@
 			(layers "*.Cu" "*.Mask")
 			(remove_unused_layers no)
-			(net "GNDA")
 		)
 		(pad "1" thru_hole circle
@@
 			)
 		)
-		(property "Value" "1N4002"
+		(property "Value" "MRA4003T3G"
 			(at 0 -2.6 0)
 			(layer "B.Fab")
@@
 		(descr "Resistor SMD 0805 (2012 Metric), square (rectangular) end terminal, IPC-7351 nominal, (Body size source: IPC-SM-782 page 72, https://www.pcb-3d.com/wordpress/wp-content/uploads/ipc-sm-782a_amendment_1_and_2.pdf)")
 		(tags "resistor")
-		(property "Reference" "R16"
+		(property "Reference" "R17"
 			(at -0.071 1.6 0)
 			(layer "B.SilkS")
@@
 			(layers "B.Cu" "B.Mask" "B.Paste")
 			(roundrect_rratio 0.243902)
-			(net "Net-(U2B-~)")
+			(net "Net-(U2A-~)")
 			(pinfunction "~_1")
 			(pintype "passive")
@@
 		(descr "Resistor SMD 0805 (2012 Metric), square (rectangular) end terminal, IPC-7351 nominal, (Body size source: IPC-SM-782 page 72, https://www.pcb-3d.com/wordpress/wp-content/uploads/ipc-sm-782a_amendment_1_and_2.pdf)")
 		(tags "resistor")
-		(property "Reference" "R19"
+		(property "Reference" "R18"
 			(at 0.0405 -1.6 0)
 			(layer "B.SilkS")
@@
 			(layers "B.Cu" "B.Mask" "B.Paste")
 			(roundrect_rratio 0.243902)
-			(net "Net-(J6-PadT)")
+			(net "Net-(J5-PadT)")
 			(pinfunction "~_1")
 			(pintype "passive")
@@
 			(layers "B.Cu" "B.Mask" "B.Paste")
 			(roundrect_rratio 0.243902)
-			(net "Net-(U2A-~)")
+			(net "Net-(U2B-~)")
 			(pinfunction "~_2")
 			(pintype "passive")
@@
 			)
 		)
-		(property "Value" "250mA"
+		(property "Value" "200mA"
 			(at 0 -1.83 90)
 			(layer "B.Fab")
@@
 			)
 		)
-		(property "Value" "1N4002"
+		(property "Value" "MRA4003T3G"
 			(at 0 -2.6 0)
 			(layer "B.Fab")
@@
 			)
 		)
-		(property "Value" "250mA"
+		(property "Value" "200mA"
 			(at 0 -1.83 90)
 			(layer "B.Fab")
@@
 		(descr "Resistor SMD 0805 (2012 Metric), square (rectangular) end terminal, IPC-7351 nominal, (Body size source: IPC-SM-782 page 72, https://www.pcb-3d.com/wordpress/wp-content/uploads/ipc-sm-782a_amendment_1_and_2.pdf)")
 		(tags "resistor")
-		(property "Reference" "R18"
+		(property "Reference" "R19"
 			(at 0.043 1.6 0)
 			(layer "B.SilkS")
@@
 			(layers "B.Cu" "B.Mask" "B.Paste")
 			(roundrect_rratio 0.243902)
-			(net "Net-(J5-PadT)")
+			(net "Net-(J6-PadT)")
 			(pinfunction "~_1")
 			(pintype "passive")
@@
 			(layers "B.Cu" "B.Mask" "B.Paste")
 			(roundrect_rratio 0.243902)
-			(net "Net-(U2B-~)")
+			(net "Net-(U2A-~)")
 			(pinfunction "~_2")
 			(pintype "passive")
@@
 		(layer "B.Cu")
 		(at 111.4 54.4 180)
-		(attr board_only exclude_from_pos_files exclude_from_bom)
 		(property "Reference" "G***"
 			(at 0 0 0)
@@
 			)
 		)
-		(attr through_hole)
+		(attr through_hole board_only exclude_from_pos_files exclude_from_bom)
 		(duplicate_pad_numbers_are_jumpers no)
 		(fp_poly
@@
 		(descr "Resistor SMD 0805 (2012 Metric), square (rectangular) end terminal, IPC-7351 nominal, (Body size source: IPC-SM-782 page 72, https://www.pcb-3d.com/wordpress/wp-content/uploads/ipc-sm-782a_amendment_1_and_2.pdf)")
 		(tags "resistor")
-		(property "Reference" "R17"
+		(property "Reference" "R16"
 			(at 0 -1.65 0)
 			(layer "B.SilkS")
@@
 			(layers "B.Cu" "B.Mask" "B.Paste")
 			(roundrect_rratio 0.243902)
-			(net "Net-(U2A-~)")
+			(net "Net-(U2B-~)")
 			(pinfunction "~_1")
 			(pintype "passive")
@@
 	)
 	(segment
-		(start 119.647 140.4)
-		(end 119.647 142.43)
+		(start 111.7555 143.7555)
+		(end 113 145)
 		(width 0.25)
 		(layer "B.Cu")
@@
 	)
 	(segment
-		(start 119.647 142.43)
-		(end 117.077 145)
+		(start 111.7555 140.4)
+		(end 111.7555 143.7555)
 		(width 0.25)
 		(layer "B.Cu")
@@
 	)
 	(segment
-		(start 111.2 140.4)
-		(end 111.2 143.2)
+		(start 119.647 142.43)
+		(end 117.077 145)
 		(width 0.25)
 		(layer "B.Cu")
@@
 	)
 	(segment
-		(start 111.2 143.2)
-		(end 113 145)
+		(start 119.647 140.4)
+		(end 119.647 142.43)
 		(width 0.25)
 		(layer "B.Cu")
@@
 	)
 	(segment
-		(start 107.175 93.0799)
-		(end 108.4549 91.8)
+		(start 108.2 126.2)
+		(end 108.6 125.8)
 		(width 0.25)
 		(layer "B.Cu")
@@
 	)
 	(segment
-		(start 110.2 88.2)
-		(end 110.3565 88.2)
+		(start 107.175 93.0799)
+		(end 108.4549 91.8)
 		(width 0.25)
 		(layer "B.Cu")
@@
 	)
 	(segment
-		(start 108.4951 94.85)
-		(end 107.5049 94.85)
+		(start 110.2 88.2)
+		(end 110.3565 88.2)
 		(width 0.25)
 		(layer "B.Cu")
@@
 	)
 	(segment
-		(start 110.319 88.1625)
-		(end 110.3565 88.2)
+		(start 109.9305 140.4)
+		(end 106.4415 140.4)
 		(width 0.25)
 		(layer "B.Cu")
@@
 	)
 	(segment
-		(start 115.975 94.625)
-		(end 108.7201 94.625)
+		(start 108.4951 94.85)
+		(end 107.5049 94.85)
 		(width 0.25)
 		(layer "B.Cu")
@@
 	)
 	(segment
-		(start 124.575 140.4)
-		(end 121.472 140.4)
+		(start 108.2 138.6695)
+		(end 108.2 126.2)
 		(width 0.25)
 		(layer "B.Cu")
@@
 	)
 	(segment
-		(start 106.6 91.8)
-		(end 110.2 88.2)
+		(start 110.319 88.1625)
+		(end 110.3565 88.2)
 		(width 0.25)
 		(layer "B.Cu")
@@
 	)
 	(segment
-		(start 106.6 92)
-		(end 106.6 91.8)
+		(start 115.975 94.625)
+		(end 108.7201 94.625)
 		(width 0.25)
 		(layer "B.Cu")
@@
 	)
 	(segment
-		(start 118.322 137.25)
-		(end 112.5049 137.25)
+		(start 106.6 91.8)
+		(end 110.2 88.2)
 		(width 0.25)
 		(layer "B.Cu")
@@
 	)
 	(segment
-		(start 112.5049 137.25)
-		(end 108.6 133.3451)
+		(start 106.6 92)
+		(end 106.6 91.8)
 		(width 0.25)
 		(layer "B.Cu")
@@
 	)
 	(segment
-		(start 121.472 140.4)
-		(end 118.322 137.25)
-		(width 0.25)
-		(layer "B.Cu")
-		(net "Net-(U2A-~)")
-	)
-	(segment
-		(start 108.6 133.3451)
-		(end 108.6 125.8)
+		(start 109.9305 140.4)
+		(end 108.2 138.6695)
 		(width 0.25)
 		(layer "B.Cu")
@@
 	)
 	(segment
-		(start 108.341116 125.175)
-		(end 108.858884 125.175)
-		(width 0.25)
-		(layer "B.Cu")
-		(net "Net-(U2B-~)")
-	)
-	(segment
 		(start 111.519 102.4)
 		(end 111.519 100.2375)
@@
 	)
 	(segment
-		(start 109.4 125.716116)
-		(end 109.4 126.6)
+		(start 119.072 138)
+		(end 112 138)
 		(width 0.25)
 		(layer "B.Cu")
@@
 	)
 	(segment
-		(start 107.975 125.541116)
-		(end 108.341116 125.175)
-		(width 0.25)
-		(layer "B.Cu")
-		(net "Net-(U2B-~)")
-	)
-	(segment
-		(start 107.975 139)
-		(end 107.975 125.541116)
-		(width 0.25)
-		(layer "B.Cu")
-		(net "Net-(U2B-~)")
-	)
-	(segment
-		(start 106.1995 140.4)
-		(end 109.375 140.4)
+		(start 111.8 104.8)
+		(end 111.519 104.519)
 		(width 0.25)
 		(layer "B.Cu")
@@
 	)
 	(segment
-		(start 111.8 104.8)
-		(end 111.519 104.519)
+		(start 112 138)
+		(end 109.4 135.4)
 		(width 0.25)
 		(layer "B.Cu")
@@
 	)
 	(segment
-		(start 109.375 140.4)
-		(end 107.975 139)
+		(start 109.4 135.4)
+		(end 109.4 126.6)
 		(width 0.25)
 		(layer "B.Cu")
@@
 	)
 	(segment
-		(start 108.858884 125.175)
-		(end 109.4 125.716116)
+		(start 121.472 140.4)
+		(end 119.072 138)
 		(width 0.25)
 		(layer "B.Cu")
@@
 		(width 0.25)
 		(layer "B.Cu")
+		(net "Net-(U2B-~)")
+	)
+	(segment
+		(start 124.575 140.4)
+		(end 121.472 140.4)
+		(width 0.25)
+		(layer "B.Cu")
