File: hardware/mixer/4ch Mixer.kicad_sch (KiCad schematic)
At the start: 56 parts, among them P1 Power, U1 TL074, U2 TL072

Commit message: Change pots to 10k (Panasonic EVU-F3AF20B14) and regenerate manufacturing files
Schematic: RV1-RV4 set to 10k, same footprint. Hand-assembly list updated with
the Panasonic part. Regenerated Gerbers, drill, placement and BOM for both boards.
Parts:
- RV1, RV2, RV3, RV4: value 100k -> 10k
Changed lines of the file:
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@@
 			)
 		)
-		(property "Value" "100k"
+		(property "Value" "10k"
 			(at 39.37 38.1 90)
 			(show_name no)
@@
 			)
 		)
-		(property "Value" "100k"
+		(property "Value" "10k"
 			(at 39.37 76.2 90)
 			(show_name no)
@@
 			)
 		)
-		(property "Value" "100k"
+		(property "Value" "10k"
 			(at 39.37 114.3 90)
 			(show_name no)
@@
 			)
 		)
-		(property "Value" "100k"
+		(property "Value" "10k"
 			(at 39.37 152.4 90)
 			(show_name no)

Commit message: Title blocks: logo worksheet, consistent company/rev across PCB and schematic
Repoint page_layout_descr_file (both pcbnew and schematic) to the real
Schenktronics worksheet path on this machine. Fill out/correct title
blocks: company standardized to "Schenktronics" (was "SchenkTronics"),
schematic rev brought from the letter "A" to "1.0" to match the real
"V1.0" silkscreen text and the new PCB title block, schematic title
aligned to "Quad Mixer" to match the board. Faceplate matched to the
same 1.0.
Other:
- company: SchenkTronics -> Schenktronics
- title: 4 Channel Active Mixer -> Quad Mixer
Changed lines of the file:
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@@
 	(paper "A")
 	(title_block
-		(title "4 Channel Active Mixer")
-		(date "2017-02-12")
-		(rev "A")
-		(company "SchenkTronics")
+		(title "Quad Mixer")
+		(date "2026-10-07")
+		(rev "1.0")
+		(company "Schenktronics")
 		(comment 1 "4 Channel Active Mixer")
 		(comment 2 "Eurorack")
