File: hardware/mixer/4ch Mixer.kicad_sch (KiCad schematic)
At the start: 56 parts, among them P1 Power, U1 TL074, U2 TL072

Commit message: Drop channel gain to ×1, swap pots to 100k, add STEP-based outline drawings
Each channel's op-amp (U1) was wired for ×2 gain, with the pot giving
0-2x overall and unity at its center click. Changed R5-R8 (feedback
resistors) from 10k to 0R, making each stage a unity-gain buffer, so
the range is now 0-1x with no gain above the input's own level. R1-R4
stay at 10k; reverting a channel to ×2 just needs its R5-R8 swapped
back to 10k. This also raises per-channel clipping headroom from
±5V to the full ±10V op-amp swing, since nothing is thrown away by a
later attenuation stage. Updated the manual, assembly guide, README,
BOM/manufacturing CSVs and the generated panel/patch drawings to
match.

Also switches RV1-RV4 from the substituted 10k pot to the originally-
specced Bourns 100k pot (no center detent), removes now-stale detent
language repo-wide, and wires in real STEP-based outline drawings
(replacing product photos in the README/manual/assembly guide).
Parts:
- R5, R6, R7, R8: value 10k -> 0
- RV1, RV2, RV3, RV4: value 10k -> 100k
Changed lines of the file:
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@@
 			)
 		)
-		(property "Value" "10k"
+		(property "Value" "0"
 			(at 82.55 50.8 90)
 			(show_name no)
@@
 			)
 		)
-		(property "Value" "10k"
+		(property "Value" "0"
 			(at 82.55 88.9 90)
 			(show_name no)
@@
 			)
 		)
-		(property "Value" "10k"
+		(property "Value" "0"
 			(at 82.55 127 90)
 			(show_name no)
@@
 			)
 		)
-		(property "Value" "10k"
+		(property "Value" "0"
 			(at 82.55 165.1 90)
 			(show_name no)
@@
 			)
 		)
-		(property "Value" "10k"
+		(property "Value" "100k"
 			(at 39.37 38.1 90)
 			(show_name no)
@@
 			)
 		)
-		(property "Value" "10k"
+		(property "Value" "100k"
 			(at 39.37 76.2 90)
 			(show_name no)
@@
 			)
 		)
-		(property "Value" "10k"
+		(property "Value" "100k"
 			(at 39.37 114.3 90)
 			(show_name no)
@@
 			)
 		)
-		(property "Value" "10k"
+		(property "Value" "100k"
 			(at 39.37 152.4 90)
 			(show_name no)
